File: ADC.kicad_sch (KiCad schematic)
At the start: 6 parts, among them Q1 2N7002, U10 CD4051B, U11 CD4051B, U12 MCP3201-BI/SN

Commit message: Update to KiCad 6
Connections:
- net ~POTI_CS renamed ~{POTI_CS}
- net ~VPOT_A3 renamed ~{VPOT_A3}
