File: Channel1-3.kicad_sch (KiCad schematic)
At the start: 53 parts, among them SW201 CH1, SW301 CH2, SW401 CH3, U201 TLC5916IDR, U202 TLC5916IDR, U301 TLC5916IDR, U401 TLC5916IDR

Commit message: Update to KiCad 6
Connections:
- net ~LED_OE renamed ~{LED_OE}
