File: Channel4-7.kicad_sch (KiCad schematic)
At the start: 68 parts, among them SW501 CH4, SW601 CH5, SW701 CH6, SW801 CH7, U501 TLC5916IDR, U601 TLC5916IDR, U701 TLC5916IDR, U801 TLC5916IDR

Commit message: Update to KiCad 6
Connections:
- net ~LED_OE renamed ~{LED_OE}
