File: Channel8-11.kicad_sch (KiCad schematic)
At the start: 68 parts, among them SW1001 CH9, SW1101 CH11, SW1201 CH11, SW901 CH8, U1001 TLC5916IDR, U1101 TLC5916IDR, U1201 TLC5916IDR, U901 TLC5916IDR

Commit message: Update to KiCad 6
Connections:
- net ~LED_OE renamed ~{LED_OE}
