File: Frontpanel.kicad_sch (KiCad schematic)
At the start: 37 parts, among them J1 FPGA, J3 Power, U1 74HC14, U3 74HC165, U4 TLC5916IDR, U5 74HC165, U7 TLC5916IDR

Commit message: Update to KiCad 6
Connections:
- net ~LED_CLK renamed ~{LED_CLK}
- net ~LED_DISPLAY_OE renamed ~{LED_DISPLAY_OE}
- net ~LED_LE renamed ~{LED_LE}
- net ~LED_OE renamed ~{LED_OE}
- net ~POTI_CS renamed ~{POTI_CS}
- net ~SW_LED_OE renamed ~{SW_LED_OE}
- net ~SW_SER_CE renamed ~{SW_SER_CE}
- net ~SW_SER_CP renamed ~{SW_SER_CP}
- net ~SW_SER_PL renamed ~{SW_SER_PL}
Other:
- sheet ADC ports: added ~{POTI_CS}; removed ~POTI_CS
- sheet Channel1-3 ports: added ~{LED_OE}; removed ~LED_OE
- sheet Channel4-7 ports: added ~{LED_OE}; removed ~LED_OE
- sheet Channel8-11 ports: added ~{LED_OE}; removed ~LED_OE
- sheet LED-Display.sch ports: added ~{LED_OE}; removed ~LED_OE
- sheet VU ports: added ~{LED_OE}; removed ~LED_OE
