File: VU.kicad_sch (KiCad schematic)
At the start: 48 parts, among them U1401 TLC5916IDR, U1402 TLC5916IDR, U1403 TLC5916IDR, U1404 TLC5916IDR

Commit message: Update to KiCad 6
Connections:
- net ~LED_OE renamed ~{LED_OE}
